File: KiCAD schematics/trotten pcb.kicad_sch (KiCad schematic)
At the start: 22 parts, among them J1 Conn_HRCU4_main, J2 Conn_screen_BRD_main, J3 Conn_screen_BRD_Slave, J4 Conn_01x04_Socket, J5 Conn_02x03_Odd_Even, M1 Motor_DC, SW1 Haut, SW2 Bas, SW3 MEM_1, SW4 MEM_2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

Commit message: commencé le moteur
Parts:
- added J7: Screw_Terminal_01x04, TerminalBlock_Phoenix:TerminalBlock_Phoenix_MPT-0,5-4-2.54_1x04_P2.54mm_Horizontal, symbol Connector:Screw_Terminal_01x04
Connections:
- net +12V: now also J7.1 (Pin_1), J7.2 (Pin_2); no longer U7.1 (IN+), U7.2 (IN+), U7.3 (IN+)
- net GND: now also J7.3 (Pin_3), J7.4 (Pin_4)
- new net: U7.1 (IN+), U7.2 (IN+), U7.3 (IN+)
- no-connect marks 20 -> 21
Changed lines of the file:
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@@
 	)
 	(junction
+		(at 208.28 127)
+		(diameter 0)
+		(color 0 0 0 0)
+	)
+	(junction
 		(at 250.19 20.32)
 		(diameter 0)
@@
 	)
 	(junction
+		(at 208.28 134.62)
+		(diameter 0)
+		(color 0 0 0 0)
+	)
+	(junction
 		(at 177.8 54.61)
 		(diameter 0)
@@
 	)
 	(no_connect
+		(at 27.94 96.52)
+	)
+	(no_connect
 		(at 212.09 46.99)
 	)
@@
 	(wire
 		(pts
+			(xy 208.28 134.62) (xy 210.82 134.62)
+		)
+		(stroke
+			(width 0)
+			(type default)
+		)
+	)
+	(wire
+		(pts
 			(xy 111.76 59.69) (xy 115.57 59.69)
 		)
@@
 	(wire
 		(pts
+			(xy 208.28 134.62) (xy 208.28 137.16)
+		)
+		(stroke
+			(width 0)
+			(type default)
+		)
+	)
+	(wire
+		(pts
 			(xy 191.77 20.32) (xy 191.77 54.61)
 		)
@@
 	(wire
 		(pts
+			(xy 208.28 127) (xy 208.28 129.54)
+		)
+		(stroke
+			(width 0)
+			(type default)
+		)
+	)
+	(wire
+		(pts
 			(xy 154.94 144.78) (xy 161.29 144.78)
 		)
@@
 	(wire
 		(pts
+			(xy 208.28 129.54) (xy 210.82 129.54)
+		)
+		(stroke
+			(width 0)
+			(type default)
+		)
+	)
+	(wire
+		(pts
 			(xy 111.76 54.61) (xy 115.57 54.61)
 		)
@@
 	(wire
 		(pts
+			(xy 208.28 132.08) (xy 208.28 134.62)
+		)
+		(stroke
+			(width 0)
+			(type default)
+		)
+	)
+	(wire
+		(pts
 			(xy 76.2 119.38) (xy 80.01 119.38)
 		)
@@
 	(wire
 		(pts
+			(xy 208.28 127) (xy 210.82 127)
+		)
+		(stroke
+			(width 0)
+			(type default)
+		)
+	)
+	(wire
+		(pts
 			(xy 111.76 67.31) (xy 130.81 67.31)
 		)
@@
 	(wire
 		(pts
+			(xy 210.82 132.08) (xy 208.28 132.08)
+		)
+		(stroke
+			(width 0)
+			(type default)
+		)
+	)
+	(wire
+		(pts
 			(xy 143.51 62.23) (xy 143.51 52.07)
 		)
@@
 	(wire
 		(pts
+			(xy 208.28 124.46) (xy 208.28 127)
+		)
+		(stroke
+			(width 0)
+			(type default)
+		)
+	)
+	(wire
+		(pts
 			(xy 190.5 77.47) (xy 190.5 59.69)
 		)
@@
 		)
 	)
-	(global_label "SCL - GP22"
-		(shape input)
-		(at 144.78 73.66 270)
-		(fields_autoplaced yes)
-		(effects
-			(font
-				(size 1.27 1.27)
-			)
-			(justify right)
-		)
-		(property "Intersheetrefs" "${INTERSHEET_REFS}"
-			(at 144.78 88.6194 90)
-			(effects
-				(font
-					(size 1.27 1.27)
-				)
-				(justify right)
-				(hide yes)
-			)
-		)
-	)
 	(global_label "L-PWM"
 		(shape input)
@@
 	(global_label "SCL - GP22"
 		(shape input)
+		(at 144.78 73.66 270)
+		(fields_autoplaced yes)
+		(effects
+			(font
+				(size 1.27 1.27)
+			)
+			(justify right)
+		)
+		(property "Intersheetrefs" "${INTERSHEET_REFS}"
+			(at 144.78 88.6194 90)
+			(effects
+				(font
+					(size 1.27 1.27)
+				)
+				(justify right)
+				(hide yes)
+			)
+		)
+	)
+	(global_label "SCL - GP22"
+		(shape input)
 		(at 95.25 105.41 90)
 		(fields_autoplaced yes)
@@
 	)
 	(symbol
+		(lib_id "Connector:Screw_Terminal_01x04")
+		(at 215.9 129.54 0)
+		(unit 1)
+		(exclude_from_sim no)
+		(in_bom yes)
+		(on_board yes)
+		(dnp no)
+		(fields_autoplaced yes)
+		(property "Reference" "J7"
+			(at 218.44 129.5399 0)
+			(effects
+				(font
+					(size 1.27 1.27)
+				)
+				(justify left)
+			)
+		)
+		(property "Value" "Screw_Terminal_01x04"
+			(at 218.44 132.0799 0)
+			(effects
+				(font
+					(size 1.27 1.27)
+				)
+				(justify left)
+			)
+		)
+		(property "Footprint" "TerminalBlock_Phoenix:TerminalBlock_Phoenix_MPT-0,5-4-2.54_1x04_P2.54mm_Horizontal"
+			(at 215.9 129.54 0)
+			(effects
+				(font
+					(size 1.27 1.27)
+				)
+				(hide yes)
+			)
+		)
+		(property "Datasheet" "~"
+			(at 215.9 129.54 0)
+			(effects
+				(font
+					(size 1.27 1.27)
+				)
+				(hide yes)
+			)
+		)
+		(property "Description" "Generic screw terminal, single row, 01x04, script generated (kicad-library-utils/schlib/autogen/connector/)"
+			(at 215.9 129.54 0)
+			(effects
+				(font
+					(size 1.27 1.27)
+				)
+				(hide yes)
+			)
+		)
+		(pin "3"
+		)
+		(pin "1"
+		)
+		(pin "4"
+		)
+		(pin "2"
+		)
+		(instances
+			(project ""
+				(path "/615cbb6f-ee23-4ea9-8e98-9b9e34f836b3"
+					(reference "J7")
+					(unit 1)
+				)
+			)
+		)
+	)
+	(symbol
 		(lib_id "HC-SR04:HC-SR04")
 		(at 139.7 175.26 0)
@@
 	)
 	(symbol
+		(lib_id "power:+12V")
+		(at 208.28 124.46 0)
+		(unit 1)
+		(exclude_from_sim no)
+		(in_bom yes)
+		(on_board yes)
+		(dnp no)
+		(fields_autoplaced yes)
+		(property "Reference" "#PWR030"
+			(at 208.28 128.27 0)
+			(effects
+				(font
+					(size 1.27 1.27)
+				)
+				(hide yes)
+			)
+		)
+		(property "Value" "+12V"
+			(at 208.28 119.38 0)
+			(effects
+				(font
+					(size 1.27 1.27)
+				)
+			)
+		)
+		(property "Footprint" ""
+			(at 208.28 124.46 0)
+			(effects
+				(font
+					(size 1.27 1.27)
+				)
+				(hide yes)
+			)
+		)
+		(property "Datasheet" ""
+			(at 208.28 124.46 0)
+			(effects
+				(font
+					(size 1.27 1.27)
+				)
+				(hide yes)
+			)
+		)
+		(property "Description" "Power symbol creates a global label with name \"+12V\""
+			(at 208.28 124.46 0)
+			(effects
+				(font
+					(size 1.27 1.27)
+				)
+				(hide yes)
+			)
+		)
+		(pin "1"
+		)
+		(instances
+			(project "trotten pcb"
+				(path "/615cbb6f-ee23-4ea9-8e98-9b9e34f836b3"
+					(reference "#PWR030")
+					(unit 1)
+				)
+			)
+		)
+	)
+	(symbol
 		(lib_id "kicad_lceda:BTS7960_SQUARE_OK")
 		(at 27.94 163.83 0)
@@
 	)
 	(symbol
-		(lib_id "power:+12V")
-		(at 27.94 96.52 0)
+		(lib_id "power:GND")
+		(at 208.28 137.16 0)
 		(unit 1)
 		(exclude_from_sim no)
@@
 		(dnp no)
 		(fields_autoplaced yes)
-		(property "Reference" "#PWR07"
-			(at 27.94 100.33 0)
+		(property "Reference" "#PWR031"
+			(at 208.28 143.51 0)
 			(effects
 				(font
@@
 			)
 		)
-		(property "Value" "+12V"
-			(at 27.94 91.44 0)
+		(property "Value" "GND"
+			(at 208.28 142.24 0)
 			(effects
 				(font
@@
 		)
 		(property "Footprint" ""
-			(at 27.94 96.52 0)
+			(at 208.28 137.16 0)
 			(effects
 				(font
@@
 		)
 		(property "Datasheet" ""
-			(at 27.94 96.52 0)
+			(at 208.28 137.16 0)
 			(effects
 				(font
@@
 			)
 		)
-		(property "Description" "Power symbol creates a global label with name \"+12V\""
-			(at 27.94 96.52 0)
+		(property "Description" "Power symbol creates a global label with name \"GND\" , ground"
+			(at 208.28 137.16 0)
 			(effects
 				(font
@@
 			(project "trotten pcb"
 				(path "/615cbb6f-ee23-4ea9-8e98-9b9e34f836b3"
-					(reference "#PWR07")
+					(reference "#PWR031")
 					(unit 1)
 				)
